File: Amon_led_board/Amon_led_board.kicad_sch (KiCad schematic)
At the start: 5 parts, among them J1 3_Pin_Male

Commit message: Update
addes new images, filled and new READMEs, added pull-ups on PCB
Other:
- note added: "RED_LED-signal WHITE_LED-signal GND"
- note removed: "RED WHITE GND"
